File: exampleLED/exampleLED.sch (KiCad schematic (older format))
At the start: 3 parts

Commit message: File to test with simulator
Other:
- note added: "Solving for R: R = 3 / .02 = 150"
- note added: "The voltage drop across the LED = 2v\n"
- note added: "The voltage drop across the resistor has to be 3v\n"
Changed lines of the file:
@@
 EESchema Schematic File Version 4
+LIBS:exampleLED-cache
 EELAYER 26 0
 EELAYER END
@@
 Text Notes 5350 2600 0    50   ~ 0
 At point B there will be 3v absolute\n
+Text Notes 5350 2700 0    50   ~ 0
+The voltage drop across the LED = 2v\n
+Text Notes 5350 2800 0    50   ~ 0
+The voltage drop across the resistor has to be 3v\n
+Text Notes 5350 2900 0    50   ~ 0
+Solving for R: R = 3 / .02 = 150
 $EndSCHEMATC
