File: theIdeaDiode/theIdeaDiode.sch (KiCad schematic (older format))
At the start: 8 parts

Commit message: :White_check_mark: More simulator work, added a voltage divider + respective tags
Parts:
- V2: value 5 -> 10
Changed lines of the file:
@@
 EESchema Schematic File Version 4
 LIBS:theIdeaDiode-cache
-EELAYER 26 0
+EELAYER 30 0
 EELAYER END
 $Descr A4 11693 8268
@@
 P 2550 4300
 F 0 "V2" H 2778 4346 50  0000 L CNN
-F 1 "5" H 2778 4255 50  0000 L CNN
+F 1 "10" H 2778 4255 50  0000 L CNN
 F 2 "" H 2550 4300 50  0001 C CNN
 F 3 "~" H 2550 4300 50  0001 C CNN
